Commit message: Updated Euler platform URDF to reflect A5 demo configuration; created moveit config package for demo configuration

File: euler_support/urdf/euler.xacro (robot description, xacro)
@@ -1,5 +1,5 @@
 <?xml version="1.0" ?>
 <robot name="euler" xmlns:xacro="http://ros.org/wiki/xacro">
-        <xacro:include filename="$(find euler_support)/urdf/euler_macro.xacro" />
-        <xacro:euler prefix=""/>
+  <xacro:include filename="$(find euler_support)/urdf/euler_macro.xacro" />
+  <xacro:euler prefix=""/>
 </robot>

File: euler_support/urdf/euler_macro.xacro (robot description, xacro)
@@ -1,173 +1,177 @@
-<?xml version="1.0" ?>
+<?xml version="1.0"?>
 <robot xmlns:xacro="http://ros.org/wiki/xacro">
-<xacro:include filename="$(find vetex_support)/urdf/vetex_macro.xacro" />
-<xacro:include filename="$(find motoman_mh5lf_support)/urdf/mh5lf_macro.xacro" />
-<!--xacro:include filename="$(find euler_support)/urdf/asus_xtion_pro.xacro" /-->
-<xacro:include filename="$(find industrial_extrinsic_cal)/urdf/asus_sensor_cal_macro.xacro" />
-<xacro:include filename="$(find euler_support)/urdf/eef_macro.xacro" />
-        <xacro:macro name="euler" params="prefix">
-        <xacro:vetex prefix="vetex_" />
-        <xacro:motoman_mh5lf prefix="motoman_" />
-        <!--xacro:asus_xtion_pro sensor_name="" off_x="0.461" off_y="0" off_z="2.103" off_rr="1.5708" off_rp="1.8849" off_ry="0"/-->
-        <xacro:asus_sensor_definitions prefix="asus" parent_link="motoman_base_link" />
-        <xacro:eef prefix=""/>
-        <!--link list -->
-        <link name="${prefix}base_link"> </link>
-	      <link name="${prefix}localization_frame"/>
-        <link name="${prefix}frame_left">
-                <visual>
-                        <origin xyz="0 0 0" rpy="0 0 0" />
-                        <geometry>
-                                <mesh filename="package://euler_support/meshes/visual/frame_left.stl" />
-                        </geometry>
-                        <material name="">
-                                <color rgba="0.752941176470588 0.752941176470588 0.752941176470588 1" />
-                        </material>
-                </visual>
-                <collision>
-                        <origin xyz="0 0 0" rpy="0 0 0" />
-                        <geometry>
-                                <mesh filename="package://euler_support/meshes/collision/frame_left.stl" />
-                        </geometry>
-                </collision>
-        </link>
-        <link name="${prefix}frame_right">
-                <visual>
-                        <origin xyz="0 0 0" rpy="0 0 0" />
-                        <geometry>
-                                <mesh filename="package://euler_support/meshes/visual/frame_right.stl" />
-                        </geometry>
-                        <material name="">
-                                <color rgba="0.752941176470588 0.752941176470588 0.752941176470588 1" />
-                        </material>
-                </visual>
-                <collision>
-                        <origin xyz="0 0 0" rpy="0 0 0" />
-                        <geometry>
-                                <mesh filename="package://euler_support/meshes/collision/frame_right.stl" />
-                        </geometry>
-                </collision>
-        </link>
-        <link name="${prefix}frame_top">
-                <visual>
-                        <origin xyz="0 0 0" rpy="0 0 0" />
-                        <geometry>
-                                <mesh filename="package://euler_support/meshes/visual/frame_top.stl" />
-                        </geometry>
-                        <material name="">
-                                <color rgba="0.752941176470588 0.752941176470588 0.752941176470588 1" />
-                        </material>
-                </visual>
-                <collision>
-                        <origin xyz="0 0 0" rpy="0 0 0" />
-                        <geometry>
-                                <mesh filename="package://euler_support/meshes/collision/frame_top.stl" />
-                        </geometry>
-                </collision>
-        </link>
-        <link name="${prefix}sick_nav350">
-                <visual>
-                        <geometry>
-                                <mesh filename="package://euler_support/meshes/visual/sick_nav350.stl" />
-                        </geometry>
-                        <material name="">
-                                <color rgba="0 0 0.752941176470588 1" />
-                        </material>
-                </visual>
-                <collision>
-                        <geometry>
-                                <mesh filename="package://euler_support/meshes/collision/sick_nav350.stl" />
-                        </geometry>
-                </collision>
-        </link>
-        <link name="${prefix}front_sick_s300">
-                <visual>
-                        <geometry>
-                                <mesh filename="package://euler_support/meshes/visual/sick_s300_mounting_assy.stl" />
-                        </geometry>
-                        <material name="">
-                                <color rgba="0.75 0.75 0 1" />
-                        </material>
-                </visual>
-                <collision>
-                        <geometry>
-                                <mesh filename="package://euler_support/meshes/collision/sick_s300_mounting_assy.stl" />
-                        </geometry>
-                </collision>
-        </link>
-        <link name="${prefix}rear_sick_s300">
-                <visual>
-                        <geometry>
-                                <mesh filename="package://euler_support/meshes/visual/sick_s300_mounting_assy.stl" />
-                        </geometry>
-                        <material name="">
-                                <color rgba="0.75 0.75 0 1" />
-                        </material>
-                </visual>
-                <collision>
-                        <geometry>
-                                <mesh filename="package://euler_support/meshes/collision/sick_s300_mounting_assy.stl" />
-                        </geometry>
-                </collision>
-        </link>
-        <joint name="${prefix}frame_left" type="fixed" >
-                <parent link="${prefix}base_link" />
-                <child link="${prefix}frame_left" />
-                <origin xyz="0 0 0" rpy="0 0 0" />
-                <axis xyz="0 0 0" />
-        </joint>
-        <joint name="${prefix}frame_right" type="fixed">
-                <parent link="${prefix}base_link" />
-                <child link="${prefix}frame_right" />
-                <origin xyz="0 0 0" rpy="0 0 0" />
-                <axis xyz="0 0 0" />
-        </joint>
-        <joint name="${prefix}frame_top" type="fixed">
-                <parent link="${prefix}base_link" />
-                <child link="${prefix}frame_top" />
-                <origin xyz="0 0 0" rpy="0 0 0" />
-                <axis xyz="0 0 0" />
-        </joint>
-        <joint name="${prefix}to_vetex" type="fixed">
-                <parent link="${prefix}base_link" />
-                <child link="${prefix}vetex_base_link" />
-                <origin xyz="0 0 0" rpy="0 0 0" />
-                <axis xyz="0 0 0" />
-        </joint>
-        <joint name="${prefix}to_arm" type="fixed">
-                <parent link="${prefix}base_link" />
-                <child link="${prefix}motoman_base_link" />
-                <origin xyz="0.067518 0 2.016" rpy="3.1415 0 0" />
-                <axis xyz="0 0 0" />
-        </joint>
-        <joint name="${prefix}sick_nav350" type="fixed">
-                <parent link="${prefix}base_link" />
-                <child link="${prefix}sick_nav350" />
-                <origin xyz="-0.239 -0.648 2.551" rpy="0 0 0" />
-                <axis xyz="0 0 0" />
-        </joint>
-        <joint name="${prefix}base_to_localization" type="fixed">
-                <parent link="${prefix}base_link" />
-                <child link="${prefix}localization_frame" />
-                <origin xyz="-0.239 -0.648 0" rpy="0 0 0" />
-                <axis xyz="0 0 0" />
-        </joint>
-        <joint name="${prefix}front_sick_s300" type="fixed">
-                <parent link="${prefix}base_link" />
-                <child link="${prefix}front_sick_s300" />
-                <origin xyz="0.193 -0.617 0.532" rpy="0 0 -0.75047" />
-                <axis xyz="0 0 0" />
-        </joint>
-        <joint name="${prefix}rear_sick_s300" type="fixed">
-                <parent link="${prefix}base_link" />
-                <child link="${prefix}rear_sick_s300" />
-                <origin xyz="-2.280 0.617 0.532" rpy="0 0  -3.96178" />
-                <axis xyz="0 0 0" />
-        </joint>
-        <joint name="motoman_link_t_to_eef_base" type="fixed">
-                <parent link="motoman_link_t" />
-                <child link="eef_base" />
-                <origin xyz="0.098 0 0" rpy="0 1.57 0" />
-        </joint>
-</xacro:macro>
+  <xacro:include filename="$(find vetex_support)/urdf/vetex_macro.xacro"/>
+  <xacro:include filename="$(find motoman_mh5lf_support)/urdf/mh5lf_macro.xacro"/>
+  <xacro:include filename="$(find euler_support)/urdf/calibration_ee_macro.xacro"/>
+<!--  <xacro:include filename="$(find flir_ptu_description)/urdf/d46.urdf.xacro"/>-->
+  <xacro:include filename="$(find localization_support)/urdf/articulated_lidar_macro.xacro"/>
+  <xacro:macro name="euler" params="prefix">
+    <xacro:vetex prefix="vetex_"/>
+    <xacro:motoman_mh5lf prefix="motoman_"/>
+    <xacro:calibration_ee prefix="calibration_ee_"/>
+    <xacro:articulated_lidar prefix="lidar_"/>
+    <!--link list -->
+    <link name="${prefix}base_link"/>
+    <link name="${prefix}localization_frame"/>
+    <link name="${prefix}frame_left">
+      <visual>
+        <origin xyz="0 0 0" rpy="0 0 0"/>
+        <geometry>
+          <mesh filename="package://euler_support/meshes/visual/frame_left.stl"/>
+        </geometry>
+        <material name="">
+          <color rgba="0.752941176470588 0.752941176470588 0.752941176470588 1"/>
+        </material>
+      </visual>
+      <collision>
+        <origin xyz="0 0 0" rpy="0 0 0"/>
+        <geometry>
+          <mesh filename="package://euler_support/meshes/collision/frame_left.stl"/>
+        </geometry>
+      </collision>
+    </link>
+    <link name="${prefix}frame_right">
+      <visual>
+        <origin xyz="0 0 0" rpy="0 0 0"/>
+        <geometry>
+          <mesh filename="package://euler_support/meshes/visual/frame_right.stl"/>
+        </geometry>
+        <material name="">
+          <color rgba="0.752941176470588 0.752941176470588 0.752941176470588 1"/>
+        </material>
+      </visual>
+      <collision>
+        <origin xyz="0 0 0" rpy="0 0 0"/>
+        <geometry>
+          <mesh filename="package://euler_support/meshes/collision/frame_right.stl"/>
+        </geometry>
+      </collision>
+    </link>
+    <link name="${prefix}frame_top">
+      <visual>
+        <origin xyz="0 0 0" rpy="0 0 0"/>
+        <geometry>
+          <mesh filename="package://euler_support/meshes/visual/frame_top.stl"/>
+        </geometry>
+        <material name="">
+          <color rgba="0.752941176470588 0.752941176470588 0.752941176470588 1"/>
+        </material>
+      </visual>
+      <collision>
+        <origin xyz="0 0 0" rpy="0 0 0"/>
+        <geometry>
+          <mesh filename="package://euler_support/meshes/collision/frame_top.stl"/>
+        </geometry>
+      </collision>
+    </link>
+    <link name="${prefix}sick_nav350">
+      <visual>
+        <geometry>
+          <mesh filename="package://euler_support/meshes/visual/sick_nav350.stl"/>
+        </geometry>
+        <material name="">
+          <color rgba="0 0 0.752941176470588 1"/>
+        </material>
+      </visual>
+      <collision>
+        <geometry>
+          <mesh filename="package://euler_support/meshes/collision/sick_nav350.stl"/>
+        </geometry>
+      </collision>
+    </link>
+    <link name="${prefix}front_sick_s300">
+      <visual>
+        <geometry>
+          <mesh filename="package://euler_support/meshes/visual/sick_s300_mounting_assy.stl"/>
+        </geometry>
+        <material name="">
+          <color rgba="0.75 0.75 0 1"/>
+        </material>
+      </visual>
+      <collision>
+        <geometry>
+          <mesh filename="package://euler_support/meshes/collision/sick_s300_mounting_assy.stl"/>
+        </geometry>
+      </collision>
+    </link>
+    <link name="${prefix}rear_sick_s300">
+      <visual>
+        <geometry>
+          <mesh filename="package://euler_support/meshes/visual/sick_s300_mounting_assy.stl"/>
+        </geometry>
+        <material name="">
+          <color rgba="0.75 0.75 0 1"/>
+        </material>
+      </visual>
+      <collision>
+        <geometry>
+          <mesh filename="package://euler_support/meshes/collision/sick_s300_mounting_assy.stl"/>
+        </geometry>
+      </collision>
+    </link>
+    <joint name="${prefix}frame_left" type="fixed">
+      <parent link="${prefix}base_link"/>
+      <child link="${prefix}frame_left"/>
+      <origin xyz="0 0 0" rpy="0 0 0"/>
+      <axis xyz="0 0 0"/>
+    </joint>
+    <joint name="${prefix}frame_right" type="fixed">
+      <parent link="${prefix}base_link"/>
+      <child link="${prefix}frame_right"/>
+      <origin xyz="0 0 0" rpy="0 0 0"/>
+      <axis xyz="0 0 0"/>
+    </joint>
+    <joint name="${prefix}frame_top" type="fixed">
+      <parent link="${prefix}base_link"/>
+      <child link="${prefix}frame_top"/>
+      <origin xyz="0 0 0" rpy="0 0 0"/>
+      <axis xyz="0 0 0"/>
+    </joint>
+    <joint name="${prefix}to_vetex" type="fixed">
+      <parent link="${prefix}base_link"/>
+      <child link="${prefix}vetex_base_link"/>
+      <origin xyz="0 0 0" rpy="0 0 0"/>
+      <axis xyz="0 0 0"/>
+    </joint>
+    <joint name="${prefix}to_arm" type="fixed">
+      <parent link="${prefix}base_link"/>
+      <child link="${prefix}motoman_base_link"/>
+      <origin xyz="0.067518 0 2.016" rpy="3.1415 0 0"/>
+      <axis xyz="0 0 0"/>
+    </joint>
+    <joint name="${prefix}sick_nav350" type="fixed">
+      <parent link="${prefix}base_link"/>
+      <child link="${prefix}sick_nav350"/>
+      <origin xyz="-0.239 -0.648 2.551" rpy="0 0 0"/>
+      <axis xyz="0 0 0"/>
+    </joint>
+    <joint name="${prefix}base_to_localization" type="fixed">
+      <parent link="${prefix}base_link"/>
+      <child link="${prefix}localization_frame"/>
+      <origin xyz="-0.239 -0.648 0" rpy="0 0 0"/>
+      <axis xyz="0 0 0"/>
+    </joint>
+    <joint name="${prefix}front_sick_s300" type="fixed">
+      <parent link="${prefix}base_link"/>
+      <child link="${prefix}front_sick_s300"/>
+      <origin xyz="0.193 -0.617 0.532" rpy="0 0 -0.75047"/>
+      <axis xyz="0 0 0"/>
+    </joint>
+    <joint name="${prefix}rear_sick_s300" type="fixed">
+      <parent link="${prefix}base_link"/>
+      <child link="${prefix}rear_sick_s300"/>
+      <origin xyz="-2.280 0.617 0.532" rpy="0 0  -3.96178"/>
+      <axis xyz="0 0 0"/>
+    </joint>
+    <joint name="${prefix}motoman_link_t_to_eef_base" type="fixed">
+      <parent link="motoman_link_t"/>
+      <child link="calibration_ee_base_link"/>
+      <origin xyz="0.098 0 0" rpy="0 ${pi/2.0} 0"/>
+    </joint>
+    <joint name="${prefix}robot_base_to_lidar" type="fixed">
+      <parent link="motoman_base_link"/>
+      <child link="lidar_base_link"/>
+      <origin xyz="-0.5 0 1.375" rpy="0 ${pi} 0"/>
+    </joint>
+  </xacro:macro>
 </robot>
