Commit message: Created new end effector xacro; created IKFast plugin for MH5; added support for dynamixel

File: euler_support/urdf/calibration_ee_new_macro.xacro (robot description, xacro)
@@ -5,5 +5,20 @@
   <xacro:property name="offset" value="${0.008 + 0.0254*sqrt((4.0**2.0)-(2.0**2.0))}"/>
   <xacro:macro name="calibration_ee_new" params="prefix">
-    <link name="${prefix}base_link"/>
+    <link name="${prefix}base_link">
+      <visual>
+        <origin xyz="0 0 0" rpy="0 0 0.005"/>
+        <geometry>
+          <cylinder length="0.010" radius="${2.25 * 0.0254}"/>
+        </geometry>
+        <material name="gray"/>
+      </visual>
+      <collision>
+        <origin xyz="0 0 0" rpy="0 0 0.005"/>
+        <geometry>
+          <cylinder length="0.010" radius="${2.25 * 0.0254}"/>
+        </geometry>
+        <material name="gray"/>
+      </collision>
+    </link>
     <link name="${prefix}tool0">
       <visual>

File: euler_support/urdf/euler_macro.xacro (robot description, xacro)
@@ -5,5 +5,6 @@
   <xacro:include filename="$(find euler_support)/urdf/calibration_ee_new_macro.xacro"/>
 <!--  <xacro:include filename="$(find flir_ptu_description)/urdf/d46.urdf.xacro"/>-->
-  <xacro:include filename="$(find localization_support)/urdf/articulated_lidar_macro.xacro"/>
+<!--  <xacro:include filename="$(find localization_support)/urdf/articulated_lidar_macro.xacro"/>-->
+  <xacro:include filename="$(find euler_support)/urdf/articulated_lidar_macro.xacro"/>
   <xacro:macro name="euler" params="prefix">
     <xacro:vetex prefix="vetex_"/>
@@ -11,5 +12,5 @@
     <xacro:calibration_ee_new prefix="calibration_ee_"/>
     <xacro:articulated_lidar prefix="lidar_"/>
-    <!--link list -->
+    <!--Link List -->
     <link name="${prefix}base_link"/>
     <link name="${prefix}localization_frame"/>
@@ -110,4 +111,5 @@
       </collision>
     </link>
+    <!-- Joint List -->
     <joint name="${prefix}frame_left" type="fixed">
       <parent link="${prefix}base_link"/>
@@ -174,5 +176,5 @@
       <parent link="motoman_base_link"/>
       <child link="lidar_base_link"/>
-      <origin xyz="-0.563283 -0.0161269 1.45662" rpy="3.12079 -0.036878 -0.0260078"/>
+      <origin xyz="-0.705989 -0.0337057 1.50329" rpy="${pi} 0 0"/>
     </joint>
   </xacro:macro>
