Commit message: Corrected innaccuracies in MH5 URDF; reformatting changes; updated numbers for calibration end effector; minor changes to articulated lidar URDF

File: euler_support/urdf/articulated_lidar_macro.xacro (robot description, xacro)
@@ -46,5 +46,5 @@
         </geometry>
         <material name="green">
-          <color rgba="0.15 0.415 0.165"/>
+          <color rgba="0.15 0.415 0.165 1"/>
         </material>
       </visual>

File: euler_support/urdf/calibration_ee_new_macro.xacro (robot description, xacro)
@@ -3,16 +3,18 @@
   <xacro:property name="r" value="${4.0*0.0254}"/>
   <xacro:property name="r_h" value="${1.8125*0.0254}"/>
-  <xacro:property name="offset" value="${0.008 + 0.0254*sqrt((4.0**2.0)-(2.0**2.0))}"/>
+<!--  <xacro:property name="offset" value="${0.008 + 0.0254*sqrt((4.0**2.0)-(2.0**2.0))}"/>-->
   <xacro:macro name="calibration_ee_new" params="prefix">
     <link name="${prefix}base_link">
       <visual>
-        <origin xyz="0 0 0" rpy="0 0 0.005"/>
+        <origin xyz="0 0 0.005" rpy="0 0 0"/>
         <geometry>
           <cylinder length="0.010" radius="${2.25 * 0.0254}"/>
         </geometry>
-        <material name="gray"/>
+        <material name="gray">
+          <color rgba="0.7 0.7 0.7 1"/>
+        </material>
       </visual>
       <collision>
-        <origin xyz="0 0 0" rpy="0 0 0.005"/>
+        <origin xyz="0 0 0.005" rpy="0 0 0"/>
         <geometry>
           <cylinder length="0.010" radius="${2.25 * 0.0254}"/>
@@ -40,5 +42,5 @@
       <parent link="${prefix}base_link"/>
       <child link="${prefix}tool0"/>
-      <origin xyz="0 0 ${offset}" rpy="0 0 0"/>
+      <origin xyz="0 0 0.095123" rpy="0 0 0"/>
     </joint>
   </xacro:macro>

File: euler_support/urdf/euler_macro.xacro (robot description, xacro)
@@ -2,5 +2,5 @@
 <robot xmlns:xacro="http://ros.org/wiki/xacro">
   <xacro:include filename="$(find vetex_support)/urdf/vetex_macro.xacro"/>
-  <xacro:include filename="$(find motoman_mh5lf_support)/urdf/mh5lf_macro.xacro"/>
+  <xacro:include filename="$(find motoman_mh5lf_support)/urdf/mh5lf_macro_formatted.xacro"/>
   <xacro:include filename="$(find euler_support)/urdf/calibration_ee_new_macro.xacro"/>
 <!--  <xacro:include filename="$(find flir_ptu_description)/urdf/d46.urdf.xacro"/>-->
@@ -169,12 +169,12 @@
     </joint>
     <joint name="${prefix}motoman_link_t_to_eef_base" type="fixed">
-      <parent link="motoman_link_t"/>
+      <parent link="motoman_tool0"/>
       <child link="calibration_ee_base_link"/>
-      <origin xyz="0.098 0 0" rpy="0 ${pi/2.0} 0"/>
+      <origin xyz="0 0 0.004" rpy="0 0 0"/>
     </joint>
     <joint name="${prefix}robot_base_to_lidar" type="fixed">
       <parent link="motoman_base_link"/>
       <child link="lidar_base_link"/>
-      <origin xyz="-0.705989 -0.0337057 1.50329" rpy="${pi} 0 0"/>
+      <origin xyz="-0.735304 0.00733868 1.47808" rpy="3.13726 -0.0149178 -0.0126956"/>
     </joint>
   </xacro:macro>

File: motoman_mh5lf_support/urdf/mh5lf.xacro (robot description, xacro)
@@ -1,5 +1,5 @@
 <?xml version="1.0" ?>
 <robot name="motoman_mh5lf" xmlns:xacro="http://ros.org/wiki/xacro">
-	<xacro:include filename="$(find motoman_mh5lf_support)/urdf/mh5lf_macro.xacro" />
-	<xacro:motoman_mh5lf prefix=""/>
+  <xacro:include filename="$(find motoman_mh5lf_support)/urdf/mh5lf_macro_formatted.xacro" />
+  <xacro:motoman_mh5lf prefix=""/>
 </robot>
