Commit message: Various changes for A5 demo compatibility

File: euler_support/urdf/euler_macro.xacro (robot description, xacro)
@@ -172,5 +172,5 @@
       <parent link="motoman_base_link"/>
       <child link="lidar_base_link"/>
-      <origin xyz="-0.5 0 1.375" rpy="0 ${pi} 0"/>
+      <origin xyz="-0.5 0 1.375" rpy="0 ${pi} ${pi}"/>
     </joint>
   </xacro:macro>

Commit message: Removed robot state publisher from moveit planning execution launch file; update URDF with 'calibrated' sensor transform; changed joint names in motoman support to work with launch structure

File: euler_support/urdf/euler_macro.xacro (robot description, xacro)
@@ -138,4 +138,5 @@
       <child link="${prefix}motoman_base_link"/>
       <origin xyz="0.067518 0 2.016" rpy="3.1415 0 0"/>
+<!--      <origin xyz="0.067518 0 2.1082" rpy="3.1415 0 0"/>-->
       <axis xyz="0 0 0"/>
     </joint>
@@ -172,5 +173,5 @@
       <parent link="motoman_base_link"/>
       <child link="lidar_base_link"/>
-      <origin xyz="-0.5 0 1.375" rpy="0 ${pi} ${pi}"/>
+      <origin xyz="-0.52599 -0.0271642 1.52919" rpy="0.0216896 -3.085 -3.1031"/>
     </joint>
   </xacro:macro>

Commit message: Moved robot up to measured height; modified link t mesh to match physical link

File: euler_support/urdf/euler_macro.xacro (robot description, xacro)
@@ -125,5 +125,6 @@
       <parent link="${prefix}base_link"/>
       <child link="${prefix}frame_top"/>
-      <origin xyz="0 0 0" rpy="0 0 0"/>
+<!--      <origin xyz="0 0 0" rpy="0 0 0"/>-->
+      <origin xyz="0 0 0.0922" rpy="0 0 0"/>
       <axis xyz="0 0 0"/>
     </joint>
@@ -137,6 +138,6 @@
       <parent link="${prefix}base_link"/>
       <child link="${prefix}motoman_base_link"/>
-      <origin xyz="0.067518 0 2.016" rpy="3.1415 0 0"/>
-<!--      <origin xyz="0.067518 0 2.1082" rpy="3.1415 0 0"/>-->
+<!--      <origin xyz="0.067518 0 2.016" rpy="3.1415 0 0"/>-->
+      <origin xyz="0.067518 0 2.1082" rpy="3.1415 0 0"/>
       <axis xyz="0 0 0"/>
     </joint>
@@ -173,5 +174,5 @@
       <parent link="motoman_base_link"/>
       <child link="lidar_base_link"/>
-      <origin xyz="-0.52599 -0.0271642 1.52919" rpy="0.0216896 -3.085 -3.1031"/>
+      <origin xyz="-0.52801 -0.0266994 1.5131" rpy="3.13392 -0.0385118 -0.0314046"/>
     </joint>
   </xacro:macro>

Commit message: Created new calibration end effector URDF

File: euler_support/urdf/euler_macro.xacro (robot description, xacro)
@@ -3,5 +3,5 @@
   <xacro:include filename="$(find vetex_support)/urdf/vetex_macro.xacro"/>
   <xacro:include filename="$(find motoman_mh5lf_support)/urdf/mh5lf_macro.xacro"/>
-  <xacro:include filename="$(find euler_support)/urdf/calibration_ee_macro.xacro"/>
+  <xacro:include filename="$(find euler_support)/urdf/calibration_ee_new_macro.xacro"/>
 <!--  <xacro:include filename="$(find flir_ptu_description)/urdf/d46.urdf.xacro"/>-->
   <xacro:include filename="$(find localization_support)/urdf/articulated_lidar_macro.xacro"/>
@@ -9,5 +9,5 @@
     <xacro:vetex prefix="vetex_"/>
     <xacro:motoman_mh5lf prefix="motoman_"/>
-    <xacro:calibration_ee prefix="calibration_ee_"/>
+    <xacro:calibration_ee_new prefix="calibration_ee_"/>
     <xacro:articulated_lidar prefix="lidar_"/>
     <!--link list -->
@@ -174,5 +174,5 @@
       <parent link="motoman_base_link"/>
       <child link="lidar_base_link"/>
-      <origin xyz="-0.52801 -0.0266994 1.5131" rpy="3.13392 -0.0385118 -0.0314046"/>
+      <origin xyz="-0.563283 -0.0161269 1.45662" rpy="3.12079 -0.036878 -0.0260078"/>
     </joint>
   </xacro:macro>

Commit message: Updated lidar position to most accurate calibration

File: euler_support/urdf/euler_macro.xacro (robot description, xacro)
@@ -176,5 +176,5 @@
       <parent link="motoman_base_link"/>
       <child link="lidar_base_link"/>
-      <origin xyz="-0.735304 0.00733868 1.47808" rpy="3.13726 -0.0149178 -0.0126956"/>
+      <origin xyz="-0.742251 0.0124948 1.46814" rpy="3.13518 -0.00343246 -0.0091254"/>
     </joint>
   </xacro:macro>

Commit message: Updated frame mesh to be one file

File: euler_support/urdf/euler_macro.xacro (robot description, xacro)
@@ -18,9 +18,9 @@
     <link name="${prefix}base_link"/>
     <link name="${prefix}localization_frame"/>
-    <link name="${prefix}frame_left">
+    <link name="${prefix}frame">
       <visual>
         <origin xyz="0 0 0" rpy="0 0 0"/>
         <geometry>
-          <mesh filename="package://euler_support/meshes/visual/frame_left.stl"/>
+          <mesh filename="package://euler_support/meshes/visual/frame.stl"/>
         </geometry>
         <material name="">
@@ -31,39 +31,5 @@
         <origin xyz="0 0 0" rpy="0 0 0"/>
         <geometry>
-          <mesh filename="package://euler_support/meshes/collision/frame_left.stl"/>
-        </geometry>
-      </collision>
-    </link>
-    <link name="${prefix}frame_right">
-      <visual>
-        <origin xyz="0 0 0" rpy="0 0 0"/>
-        <geometry>
-          <mesh filename="package://euler_support/meshes/visual/frame_right.stl"/>
-        </geometry>
-        <material name="">
-          <color rgba="0.752941176470588 0.752941176470588 0.752941176470588 1"/>
-        </material>
-      </visual>
-      <collision>
-        <origin xyz="0 0 0" rpy="0 0 0"/>
-        <geometry>
-          <mesh filename="package://euler_support/meshes/collision/frame_right.stl"/>
-        </geometry>
-      </collision>
-    </link>
-    <link name="${prefix}frame_top">
-      <visual>
-        <origin xyz="0 0 0" rpy="0 0 0"/>
-        <geometry>
-          <mesh filename="package://euler_support/meshes/visual/frame_top.stl"/>
-        </geometry>
-        <material name="">
-          <color rgba="0.752941176470588 0.752941176470588 0.752941176470588 1"/>
-        </material>
-      </visual>
-      <collision>
-        <origin xyz="0 0 0" rpy="0 0 0"/>
-        <geometry>
-          <mesh filename="package://euler_support/meshes/collision/frame_top.stl"/>
+          <mesh filename="package://euler_support/meshes/collision/frame.stl"/>
         </geometry>
       </collision>
@@ -114,21 +80,7 @@
       </collision>
     </link>
-    <joint name="${prefix}frame_left" type="fixed">
+    <joint name="${prefix}frame_to_platform" type="fixed">
       <parent link="${prefix}base_link"/>
-      <child link="${prefix}frame_left"/>
-      <origin xyz="0 0 0" rpy="0 0 0"/>
-      <axis xyz="0 0 0"/>
-    </joint>
-    <joint name="${prefix}frame_right" type="fixed">
-      <parent link="${prefix}base_link"/>
-      <child link="${prefix}frame_right"/>
-      <origin xyz="0 0 0" rpy="0 0 0"/>
-      <axis xyz="0 0 0"/>
-    </joint>
-    <joint name="${prefix}frame_top" type="fixed">
-      <parent link="${prefix}base_link"/>
-      <child link="${prefix}frame_top"/>
-      <origin xyz="0 0 0" rpy="0 0 0"/>
-      <axis xyz="0 0 0"/>
+      <child link="${prefix}frame"/>
     </joint>
     <joint name="${prefix}to_vetex" type="fixed">
