Commit message: test

File: motoman_mh5lf_support/urdf/mh5lf_macro_formatted.xacro (robot description, xacro)
@@ -1,4 +1,5 @@
 <?xml version="1.0"?>
 <robot xmlns:xacro="http://ros.org/wiki/xacro">
+  <xacro:property name="base_offset" value="0.330"/>
   <xacro:macro name="motoman_mh5lf" params="prefix">
     <!-- link list -->
@@ -6,4 +7,5 @@
     <link name="${prefix}base_link">
       <visual>
+        <origin rpy="0 0 0"/>
         <geometry>
           <mesh filename="package://motoman_mh5lf_support/meshes/mh5lf/visual/base_link.stl"/>
@@ -14,4 +16,5 @@
       </visual>
       <collision>
+        <origin rpy="0 0 0"/>
         <geometry>
           <mesh filename="package://motoman_mh5lf_support/meshes/mh5lf/collision/base_link.stl"/>
@@ -108,5 +111,4 @@
       </collision>
     </link>
-    <link name="${prefix}tool0"/>
     <!-- end of link list -->
     <!-- joint list -->
@@ -114,52 +116,47 @@
       <parent link="${prefix}base_link"/>
       <child link="${prefix}link_s"/>
-      <origin xyz="0 0 0.330" rpy="0 0 0"/>
+      <origin xyz="0 0 0" rpy="0 0 0"/>
       <axis xyz="0 0 1"/>
-      <limit lower="-${radians(170)}" upper="${radians(170)}" effort="100" velocity="${radians(270)}"/>
+      <limit lower="-2.96697222222222" upper="2.96697222222222" effort="100" velocity="4.71225"/>
+    </joint>
+    <joint name="${prefix}base_to_base_software" type="fixed">
+      <parent link="${prefix}base_link"/>
+      <child link="${prefix}base_software"/>
+      <origin xyz="0 0 ${base_offset}" rpy="0 0 0"/>
     </joint>
     <joint name="${prefix}joint_l" type="revolute">
       <parent link="${prefix}link_s"/>
       <child link="${prefix}link_l"/>
-      <origin xyz="0.088 0 0" rpy="0 0 0"/>
+      <origin xyz="0.088 0 0.36" rpy="0 0 0"/>
       <axis xyz="0 1 0"/>
-      <limit lower="-${radians(65)}" upper="${radians(150)}" effort="100" velocity="${radians(280)}"/>
+      <limit lower="-1.13443055555556" upper="2.61791666666667" effort="100" velocity="4.88677777777778"/>
     </joint>
     <joint name="${prefix}joint_u" type="revolute">
       <parent link="${prefix}link_l"/>
       <child link="${prefix}link_u"/>
-      <origin xyz="0 0 0.400" rpy="0 0 0"/>
+      <origin xyz="0 0 0.4" rpy="0 0 0"/>
       <axis xyz="0 -1 0"/>
-      <limit lower="-${radians(138)}" upper="${radians(255)}" effort="100" velocity="${radians(300)}"/>
+      <limit lower="-2.40848333333333" upper="4.45045833333333" effort="100" velocity="5.23583333333333"/>
     </joint>
     <joint name="${prefix}joint_r" type="revolute">
       <parent link="${prefix}link_u"/>
       <child link="${prefix}link_r"/>
-      <origin xyz="0 0 0.040" rpy="0 0 0"/>
+      <origin xyz="0 0 0.04" rpy="0 0 0"/>
       <axis xyz="-1 0 0"/>
-      <limit lower="-${radians(190)}" upper="${radians(190)}" effort="100" velocity="${radians(450)}"/>
+      <limit lower="-3.31602777777778" upper="3.31602777777778" effort="100" velocity="7.85375"/>
     </joint>
     <joint name="${prefix}joint_b" type="revolute">
       <parent link="${prefix}link_r"/>
       <child link="${prefix}link_b"/>
-      <origin xyz="0.405 0 0" rpy="0 0 0"/>
+      <origin xyz="0.404 0 0" rpy="0 0 0"/>
       <axis xyz="0 -1 0"/>
-      <limit lower="-${radians(135)}" upper="${radians(135)}" effort="100" velocity="${radians(450)}"/>
+      <limit lower="-2.356125" upper="2.356125" effort="100" velocity="7.85375"/>
     </joint>
     <joint name="${prefix}joint_t" type="revolute">
       <parent link="${prefix}link_b"/>
       <child link="${prefix}link_t"/>
-      <origin xyz="0.080 0 0" rpy="0 0 0"/>
+      <origin xyz="0 0 0" rpy="0 0 0"/>
       <axis xyz="-1 0 0"/>
-      <limit lower="-${radians(360)}" upper="${radians(360)}" effort="100" velocity="${radians(720)}"/>
-    </joint>
-    <joint name="${prefix}joint_t_tool0" type="fixed">
-      <parent link="${prefix}link_t"/>
-      <child link="${prefix}tool0"/>
-      <origin xyz="0 0 0" rpy="0 ${radians(90)} 0"/>
-    </joint>
-    <joint name="${prefix}base_to_base_software" type="fixed">
-      <parent link="${prefix}base_link"/>
-      <child link="${prefix}base_software"/>
-      <origin xyz="0 0 0.330" rpy="0 0 0"/>
+      <limit lower="-6.283" upper="6.283" effort="100" velocity="12.566"/>
     </joint>
     <!-- end of joint list -->
